File: KiCAD/KiCAD.kicad_pcb (KiCad board)
At the start: 2 copper layers, 90 x 94 mm, 20 parts, among them M2_1 MountingHole_2.2mm_M2, M2_2 MountingHole_2.2mm_M2, M2_3 MountingHole_2.2mm_M2, M2_4 MountingHole_2.2mm_M2, SW1 SW_Push, SW10 RotaryEncoder_Switch, SW11 RotaryEncoder_Switch, SW2 SW_Push, SW3 SW_Push, SW4 SW_Push, SW5 SW_Push, SW6 SW_Push, SW7 SW_Push, SW8 SW_Push, SW9 RotaryEncoder_Switch

Commit message: miaw
Parts:
- moved ME1 14.0 mm to (215.6, 101.6)
- moved RV1 14.0 mm to (215.6, 87.6)
Connections:
- A1 pad 25: Net-(A1-GPIO19) -> unconnected-(A1-GPIO19-Pad25)
- A1 pad 34: unconnected-(A1-GPIO28_ADC2-Pad34) -> Net-(A1-GPIO28_ADC2)
- RV1 pad 2: Net-(A1-GPIO19) -> Net-(A1-GPIO28_ADC2)
Routing:
- net Net-(A1-GPIO28_ADC2): track 0.00 -> 35.1 mm
- net Net-(A1-GPIO19): track 18.2 -> 0.00 mm
- net Net-(A1-3V3): track 177.5 -> 189.9 mm
- net Net-(A1-GPIO26_ADC0): track 16.7 -> 22.5 mm
Changed lines of the file:
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@@
 	(net 6 "Net-(A1-GPIO5)")
 	(net 7 "Net-(A1-GPIO8)")
-	(net 8 "unconnected-(A1-GPIO28_ADC2-Pad34)")
+	(net 8 "unconnected-(A1-GPIO19-Pad25)")
 	(net 9 "Net-(A1-GPIO16)")
 	(net 10 "unconnected-(A1-GND-Pad13)_1")
@@
 	(net 19 "Net-(A1-GPIO14)")
 	(net 20 "Net-(A1-GPIO9)")
-	(net 21 "Net-(A1-GPIO19)")
+	(net 21 "Net-(A1-GPIO28_ADC2)")
 	(net 22 "unconnected-(A1-3V3_EN-Pad37)")
 	(net 23 "unconnected-(A1-ADC_VREF-Pad35)")
@@
 			(layers "*.Cu" "*.Mask")
 			(remove_unused_layers no)
-			(net 21 "Net-(A1-GPIO19)")
+			(net 8 "unconnected-(A1-GPIO19-Pad25)")
 			(pinfunction "GPIO19")
-			(pintype "bidirectional")
+			(pintype "bidirectional+no_connect")
 		)
 		(pad "26" thru_hole circle
@@
 			(layers "*.Cu" "*.Mask")
 			(remove_unused_layers no)
-			(net 8 "unconnected-(A1-GPIO28_ADC2-Pad34)")
+			(net 21 "Net-(A1-GPIO28_ADC2)")
 			(pinfunction "GPIO28_ADC2")
-			(pintype "bidirectional+no_connect")
+			(pintype "bidirectional")
 		)
 		(pad "35" thru_hole circle
@@
 	(footprint "Connector_Wire:SolderWire-0.5sqmm_1x03_P4.6mm_D0.9mm_OD2.1mm_Relief"
 		(layer "F.Cu")
-		(at 215.59 87.6 90)
+		(at 215.59 101.6 90)
 		(descr "Soldered wire connection with feed through strain relief, for 3 times 0.5 mm² wires, basic insulation, conductor diameter 0.9mm, outer diameter 2.1mm, size source Multi-Contact FLEXI-E 0.50 (https://www.staubli.com/content/dam/ecs/catalogs-brochures/TM/CAB-Main-11014119-en.pdf#page=9), bend radius 3 times outer diameter, generated with kicad-footprint-generator")
 		(tags "connector wire 0.5sqmm strain-relief")
@@
 	(footprint "Connector_Wire:SolderWire-0.5sqmm_1x03_P4.6mm_D0.9mm_OD2.1mm_Relief"
 		(layer "F.Cu")
-		(at 215.59 101.6 90)
+		(at 215.59 87.6 90)
 		(descr "Soldered wire connection with feed through strain relief, for 3 times 0.5 mm² wires, basic insulation, conductor diameter 0.9mm, outer diameter 2.1mm, size source Multi-Contact FLEXI-E 0.50 (https://www.staubli.com/content/dam/ecs/catalogs-brochures/TM/CAB-Main-11014119-en.pdf#page=9), bend radius 3 times outer diameter, generated with kicad-footprint-generator")
 		(tags "connector wire 0.5sqmm strain-relief")
@@
 			(layers "*.Cu" "*.Mask")
 			(remove_unused_layers no)
-			(net 21 "Net-(A1-GPIO19)")
+			(net 21 "Net-(A1-GPIO28_ADC2)")
 			(pinfunction "2")
 			(pintype "passive")
@@
 	)
 	(segment
+		(start 221.5 67.3)
+		(end 217.88 67.3)
+		(width 0.254)
+		(layer "F.Cu")
+		(net 11)
+	)
+	(segment
 		(start 179.4 60)
 		(end 201.6 60)
@@
 	)
 	(segment
-		(start 174.6 55.2)
-		(end 179.4 60)
+		(start 206.6 69.4)
+		(end 215.78 69.4)
 		(width 0.254)
 		(layer "F.Cu")
@@
 	)
 	(segment
-		(start 221.89 76.7)
-		(end 221.89 86.1)
+		(start 174.6 55.2)
+		(end 179.4 60)
 		(width 0.254)
 		(layer "F.Cu")
@@
 	)
 	(segment
-		(start 152.8 65.4)
-		(end 152.8 60.5)
+		(start 221.5 67.3)
+		(end 221.5 75.12)
 		(width 0.254)
 		(layer "F.Cu")
@@
 	)
 	(segment
-		(start 221.89 86.1)
-		(end 215.59 92.4)
+		(start 152.8 65.4)
+		(end 152.8 60.5)
 		(width 0.254)
 		(layer "F.Cu")
@@
 	)
 	(segment
-		(start 211.305 73.875)
-		(end 215.78 69.4)
+		(start 229.9 67.3)
+		(end 221.5 67.3)
 		(width 0.254)
 		(layer "F.Cu")
@@
 	)
 	(segment
-		(start 229.9 67.3)
-		(end 217.88 67.3)
+		(start 215.59 78.4)
+		(end 212.4 81.59)
 		(width 0.254)
 		(layer "F.Cu")
@@
 	)
 	(segment
-		(start 221.89 76.7)
-		(end 215.59 83)
+		(start 199.3 73.82)
+		(end 202.18 73.82)
+		(width 0.254)
+		(layer "F.Cu")
+		(net 11)
+	)
+	(segment
+		(start 212.4 84.1)
+		(end 213.4 85.1)
 		(width 0.254)
 		(layer "F.Cu")
@@
 	)
 	(segment
+		(start 213.4 85.1)
+		(end 221.89 85.1)
+		(width 0.254)
+		(layer "F.Cu")
+		(net 11)
+	)
+	(segment
+		(start 221.5 75.12)
+		(end 221.9 75.52)
+		(width 0.254)
+		(layer "F.Cu")
+		(net 11)
+	)
+	(segment
 		(start 202.9 62.4)
 		(end 229.5 62.4)
@@
 	)
 	(segment
-		(start 199.34 73.875)
-		(end 211.305 73.875)
+		(start 215.59 97)
+		(end 221.89 90.7)
 		(width 0.254)
 		(layer "F.Cu")
@@
 	)
 	(segment
-		(start 215.78 69.4)
-		(end 221.9 75.52)
+		(start 212.4 81.59)
+		(end 212.4 84.1)
 		(width 0.254)
 		(layer "F.Cu")
@@
 	)
 	(segment
+		(start 221.89 90.7)
+		(end 221.89 85.1)
+		(width 0.254)
+		(layer "F.Cu")
+		(net 11)
+	)
+	(segment
 		(start 231.2 66)
 		(end 229.9 67.3)
@@
 	)
 	(segment
+		(start 221.89 85.1)
+		(end 221.89 76.7)
+		(width 0.254)
+		(layer "F.Cu")
+		(net 11)
+	)
+	(segment
 		(start 201.6 60)
 		(end 201.6 61.1)
@@
 	)
 	(segment
+		(start 202.18 73.82)
+		(end 206.6 69.4)
+		(width 0.254)
+		(layer "F.Cu")
+		(net 11)
+	)
+	(segment
 		(start 158.1 55.2)
 		(end 174.6 55.2)
@@
 	)
 	(segment
-		(start 215.59 87.6)
-		(end 200.365 87.6)
+		(start 199.34 86.575)
+		(end 214.365 101.6)
 		(width 0.254)
 		(layer "F.Cu")
@@
 	)
 	(segment
-		(start 200.365 87.6)
-		(end 199.34 86.575)
+		(start 214.365 101.6)
+		(end 215.59 101.6)
 		(width 0.254)
 		(layer "F.Cu")
@@
 	)
 	(segment
-		(start 215.59 97)
-		(end 210.775 101.815)
+		(start 218.8 79.79)
+		(end 215.59 83)
+		(width 0.254)
+		(layer "F.Cu")
+		(net 21)
+	)
+	(segment
+		(start 218.8 71.7)
+		(end 218.8 79.79)
+		(width 0.254)
+		(layer "F.Cu")
+		(net 21)
+	)
+	(segment
+		(start 199.3 78.9)
+		(end 206.5 71.7)
 		(width 0.254)
 		(layer "F.Cu")
@@
 	)
 	(segment
-		(start 210.775 101.815)
-		(end 199.34 101.815)
+		(start 206.5 71.7)
+		(end 218.8 71.7)
 		(width 0.254)
 		(layer "F.Cu")

Commit message: f
Routing:
- net Net-(A1-GPIO15): track 36.6 -> 27.2 mm
- net Net-(A1-GPIO13): track 33.6 -> 27.0 mm
- net Net-(A1-GPIO14): track 31.2 -> 25.5 mm
- net Net-(A1-GPIO12): track 28.0 -> 23.3 mm
- net Net-(A1-GPIO7): track 41.7 -> 44.3 mm
- net Net-(A1-GPIO4): track 33.6 -> 35.8 mm
- net Net-(A1-GPIO11): track 30.1 -> 28.1 mm
- net Net-(A1-GPIO6): track 35.5 -> 36.7 mm
- net Net-(A1-GPIO9): track 41.9 -> 43.0 mm
- net Net-(A1-GPIO3): track 25.3 -> 26.3 mm
